Commit message: fully actuated example functional, work in progress for real pisa hand sensorised

File: examples/full_actuated_example/robot/soft_hand_full_actuation.urdf.xacro (robot description, xacro)
@@ -24,5 +24,5 @@
 	</gazebo>
 	<xacro:soft_hand parent="box" name="soft_hand" left="false" withAdaptiveTransmission="false" useMimicTag="$(arg use_mimic_tag)">
-		<origin xyz="0.002 0.009 0.038" rpy="0 0 0"/>
+		<origin xyz="0.0 0.0 1.02" rpy="0 0 0"/>
 	</xacro:soft_hand>
 </robot>

File: soft_hand_description/model/soft_hand.transmission.xacro (robot description, xacro)
@@ -1,4 +1,7 @@
 <?xml version="1.0"?>
 <robot name="robot" xmlns:xacro="http://www.ros.org/wiki/xacro">
+    <xacro:property name="Interface30" value="hardware_interface/PositionJointInterface"/>
+		<xacro:property name="Interface10" value="hardware_interface/PositionJointInterface"/>
+    <xacro:property name="Interface40" value="hardware_interface/EffortJointInterface"/>
     <xacro:macro name="finger_transmission" params="name finger">
         <transmission name="${name}_${finger}_abd_trans">
@@ -6,5 +9,6 @@
         <type>transmission_interface/SimpleTransmission</type>
         <joint name="${name}_${finger}_abd_joint">
-          <hardwareInterface>EffortJointInterface</hardwareInterface>
+          <!--hardwareInterface>hardware_interface/PositionJointInterface</hardwareInterface-->
+          <hardwareInterface>${Interface10}</hardwareInterface>
         </joint>
         <actuator name="${name}_${finger}_abd_motor">
@@ -16,5 +20,6 @@
         <type>transmission_interface/SimpleTransmission</type>
         <joint name="${name}_${finger}_inner_joint">
-          <hardwareInterface>EffortJointInterface</hardwareInterface>
+          <!--hardwareInterface>hardware_interface/PositionJointInterface</hardwareInterface-->
+          <hardwareInterface>${Interface10}</hardwareInterface>
         </joint>
         <actuator name="${name}_${finger}_inner_motor">
@@ -26,5 +31,6 @@
         <type>transmission_interface/SimpleTransmission</type>
         <joint name="${name}_${finger}_inner_joint_mimic">
-          <hardwareInterface>EffortJointInterface</hardwareInterface>
+          <!--hardwareInterface>hardware_interface/PositionJointInterface</hardwareInterface-->
+          <hardwareInterface>${Interface10}</hardwareInterface>
         </joint>
         <actuator name="${name}_${finger}_inner_motor">
@@ -36,5 +42,6 @@
         <type>transmission_interface/SimpleTransmission</type>
         <joint name="${name}_${finger}_middle_joint">
-          <hardwareInterface>EffortJointInterface</hardwareInterface>
+          <!--hardwareInterface>hardware_interface/PositionJointInterface</hardwareInterface-->
+          <hardwareInterface>${Interface10}</hardwareInterface>
         </joint>
         <actuator name="${name}_${finger}_middle_motor">
@@ -46,5 +53,6 @@
         <type>transmission_interface/SimpleTransmission</type>
         <joint name="${name}_${finger}_middle_joint_mimic">
-          <hardwareInterface>EffortJointInterface</hardwareInterface>
+          <!--hardwareInterface>hardware_interface/PositionJointInterface</hardwareInterface-->
+          <hardwareInterface>${Interface10}</hardwareInterface>
         </joint>
         <actuator name="${name}_${finger}_middle_motor">
@@ -56,5 +64,6 @@
         <type>transmission_interface/SimpleTransmission</type>
         <joint name="${name}_${finger}_outer_joint">
-          <hardwareInterface>EffortJointInterface</hardwareInterface>
+          <!--hardwareInterface>hardware_interface/PositionJointInterface</hardwareInterface-->
+          <hardwareInterface>${Interface10}</hardwareInterface>
         </joint>
         <actuator name="${name}_${finger}_outer_motor">
@@ -66,5 +75,6 @@
         <type>transmission_interface/SimpleTransmission</type>
         <joint name="${name}_${finger}_outer_joint_mimic">
-          <hardwareInterface>EffortJointInterface</hardwareInterface>
+          <!--hardwareInterface>hardware_interface/PositionJointInterface</hardwareInterface-->
+          <hardwareInterface>${Interface10}</hardwareInterface>
         </joint>
         <actuator name="${name}_${finger}_outer_motor">
@@ -79,5 +89,6 @@
           <type>transmission_interface/SimpleTransmission</type>
           <joint name="${name}_thumb_abd_joint">
-            <hardwareInterface>EffortJointInterface</hardwareInterface>
+            <!--hardwareInterface>hardware_interface/PositionJointInterface</hardwareInterface-->
+            <hardwareInterface>${Interface10}</hardwareInterface>
           </joint>
           <actuator name="${name}_thumb_abd_motor">
@@ -89,5 +100,6 @@
           <type>transmission_interface/SimpleTransmission</type>
           <joint name="${name}_thumb_inner_joint">
-            <hardwareInterface>EffortJointInterface</hardwareInterface>
+            <!--hardwareInterface>hardware_interface/PositionJointInterface</hardwareInterface-->
+            <hardwareInterface>${Interface10}</hardwareInterface>
           </joint>
           <actuator name="${name}_thumb_inner_motor">
@@ -99,5 +111,6 @@
           <type>transmission_interface/SimpleTransmission</type>
           <joint name="${name}_thumb_inner_joint_mimic">
-            <hardwareInterface>EffortJointInterface</hardwareInterface>
+          <!--hardwareInterface>hardware_interface/PositionJointInterface</hardwareInterface-->
+            <hardwareInterface>${Interface10}</hardwareInterface>
           </joint>
           <actuator name="${name}_thumb_inner_motor">
@@ -109,5 +122,6 @@
           <type>transmission_interface/SimpleTransmission</type>
           <joint name="${name}_thumb_outer_joint">
-            <hardwareInterface>EffortJointInterface</hardwareInterface>
+          <!--hardwareInterface>hardware_interface/PositionJointInterface</hardwareInterface-->
+            <hardwareInterface>${Interface10}</hardwareInterface>
           </joint>
           <actuator name="${name}_thumb_outer_motor">
@@ -119,5 +133,6 @@
           <type>transmission_interface/SimpleTransmission</type>
           <joint name="${name}_thumb_outer_joint_mimic">
-            <hardwareInterface>EffortJointInterface</hardwareInterface>
+          <!--hardwareInterface>hardware_interface/PositionJointInterface</hardwareInterface-->
+            <hardwareInterface>${Interface10}</hardwareInterface>
           </joint>
           <actuator name="${name}_thumb_outer_motor">
@@ -136,6 +151,7 @@
           <type>transmission_interface/SimpleTransmission</type>
           <joint name="${name}_synergy_joint">
-            <hardwareInterface>PositionJointInterface</hardwareInterface>
-            <!--hardwareInterface>EffortJointInterface</hardwareInterface-->
+            <!-- <hardwareInterface>hardware_interface/PositionJointInterface</hardwareInterface> -->
+            <hardwareInterface>${Interface30}</hardwareInterface>
+            <!-- <hardwareInterface>${Interface10}</hardwareInterface> -->
           </joint>
           <actuator name="${name}_synergy_motor">
@@ -151,6 +167,6 @@
             <mechanicalReduction>1.3</mechanicalReduction>
             <mechanicalElasticity>1.0</mechanicalElasticity>
-            <!-- hardwareInterface>PositionJointInterface</hardwareInterface -->
-            <hardwareInterface>EffortJointInterface</hardwareInterface>
+            <!--hardwareInterface>hardware_interface/PositionJointInterface</hardwareInterface-->
+            <hardwareInterface>${Interface10}</hardwareInterface>
           </joint>
           <joint name="${name}_thumb_inner_joint">
@@ -159,6 +175,6 @@
             <mechanicalReduction>1.0</mechanicalReduction>
             <mechanicalElasticity>1.0</mechanicalElasticity>
-            <!-- hardwareInterface>PositionJointInterface</hardwareInterface -->
-            <hardwareInterface>EffortJointInterface</hardwareInterface>
+            <!--hardwareInterface>hardware_interface/PositionJointInterface</hardwareInterface-->
+            <hardwareInterface>${Interface10}</hardwareInterface>
           </joint>
           <joint name="${name}_thumb_outer_joint">
@@ -167,6 +183,6 @@
             <mechanicalReduction>1.0</mechanicalReduction>
             <mechanicalElasticity>1.0</mechanicalElasticity>
-            <!-- hardwareInterface>PositionJointInterface</hardwareInterface -->
-            <hardwareInterface>EffortJointInterface</hardwareInterface>
+            <!--hardwareInterface>hardware_interface/PositionJointInterface</hardwareInterface-->
+            <hardwareInterface>${Interface10}</hardwareInterface>
           </joint>
           <joint name="${name}_index_abd_joint">
@@ -175,6 +191,6 @@
             <mechanicalReduction>-0.2</mechanicalReduction>
             <mechanicalElasticity>1.0</mechanicalElasticity>
-            <!-- hardwareInterface>PositionJointInterface</hardwareInterface -->
-            <hardwareInterface>EffortJointInterface</hardwareInterface>
+            <!--hardwareInterface>hardware_interface/PositionJointInterface</hardwareInterface-->
+            <hardwareInterface>${Interface10}</hardwareInterface>
           </joint>
           <joint name="${name}_index_inner_joint">
@@ -183,6 +199,6 @@
             <mechanicalReduction>1.0</mechanicalReduction>
             <mechanicalElasticity>1.0</mechanicalElasticity>
-            <!-- hardwareInterface>PositionJointInterface</hardwareInterface -->
-            <hardwareInterface>EffortJointInterface</hardwareInterface>
+            <!--hardwareInterface>hardware_interface/PositionJointInterface</hardwareInterface-->
+            <hardwareInterface>${Interface10}</hardwareInterface>
           </joint>
           <joint name="${name}_index_middle_joint">
@@ -191,6 +207,6 @@
             <mechanicalReduction>1.0</mechanicalReduction>
             <mechanicalElasticity>1.0</mechanicalElasticity>
-            <!-- hardwareInterface>PositionJointInterface</hardwareInterface -->
-            <hardwareInterface>EffortJointInterface</hardwareInterface>
+            <!--hardwareInterface>hardware_interface/PositionJointInterface</hardwareInterface-->
+            <hardwareInterface>${Interface10}</hardwareInterface>
           </joint>
           <joint name="${name}_index_outer_joint">
@@ -199,6 +215,6 @@
             <mechanicalReduction>1.0</mechanicalReduction>
             <mechanicalElasticity>1.0</mechanicalElasticity>
-            <!-- hardwareInterface>PositionJointInterface</hardwareInterface -->
-            <hardwareInterface>EffortJointInterface</hardwareInterface>
+            <!--hardwareInterface>hardware_interface/PositionJointInterface</hardwareInterface-->
+            <hardwareInterface>${Interface10}</hardwareInterface>
           </joint>
           <joint name="${name}_middle_abd_joint">
@@ -207,6 +223,6 @@
             <mechanicalReduction>0.001</mechanicalReduction>
             <mechanicalElasticity>1.0</mechanicalElasticity>
-            <!-- hardwareInterface>PositionJointInterface</hardwareInterface -->
-            <hardwareInterface>EffortJointInterface</hardwareInterface>
+            <!--hardwareInterface>hardware_interface/PositionJointInterface</hardwareInterface-->
+            <hardwareInterface>${Interface10}</hardwareInterface>
           </joint>
           <joint name="${name}_middle_inner_joint">
@@ -215,6 +231,6 @@
             <mechanicalReduction>1.0</mechanicalReduction>
             <mechanicalElasticity>1.0</mechanicalElasticity>
-            <!-- hardwareInterface>PositionJointInterface</hardwareInterface -->
-            <hardwareInterface>EffortJointInterface</hardwareInterface>
+            <!--hardwareInterface>hardware_interface/PositionJointInterface</hardwareInterface-->
+            <hardwareInterface>${Interface10}</hardwareInterface>
           </joint>
           <joint name="${name}_middle_middle_joint">
@@ -223,6 +239,6 @@
             <mechanicalReduction>1.0</mechanicalReduction>
             <mechanicalElasticity>1.0</mechanicalElasticity>
-            <!-- hardwareInterface>PositionJointInterface</hardwareInterface -->
-            <hardwareInterface>EffortJointInterface</hardwareInterface>
+            <!--hardwareInterface>hardware_interface/PositionJointInterface</hardwareInterface-->
+            <hardwareInterface>${Interface10}</hardwareInterface>
           </joint>
           <joint name="${name}_middle_outer_joint">
@@ -231,6 +247,6 @@
             <mechanicalReduction>1.0</mechanicalReduction>
             <mechanicalElasticity>1.0</mechanicalElasticity>
-            <!-- hardwareInterface>PositionJointInterface</hardwareInterface -->
-            <hardwareInterface>EffortJointInterface</hardwareInterface>
+            <!--hardwareInterface>hardware_interface/PositionJointInterface</hardwareInterface-->
+            <hardwareInterface>${Interface10}</hardwareInterface>
           </joint>
           <joint name="${name}_ring_abd_joint">
@@ -239,6 +255,6 @@
             <mechanicalReduction>0.2</mechanicalReduction>
             <mechanicalElasticity>1.0</mechanicalElasticity>
-            <!-- hardwareInterface>PositionJointInterface</hardwareInterface -->
-            <hardwareInterface>EffortJointInterface</hardwareInterface>
+            <!--hardwareInterface>hardware_interface/PositionJointInterface</hardwareInterface-->
+            <hardwareInterface>${Interface10}</hardwareInterface>
           </joint>
           <joint name="${name}_ring_inner_joint">
@@ -247,6 +263,6 @@
             <mechanicalReduction>1.0</mechanicalReduction>
             <mechanicalElasticity>1.0</mechanicalElasticity>
-            <!-- hardwareInterface>PositionJointInterface</hardwareInterface -->
-            <hardwareInterface>EffortJointInterface</hardwareInterface>
+            <!--hardwareInterface>hardware_interface/PositionJointInterface</hardwareInterface-->
+            <hardwareInterface>${Interface10}</hardwareInterface>
           </joint>
           <joint name="${name}_ring_middle_joint">
@@ -255,6 +271,6 @@
             <mechanicalReduction>1.0</mechanicalReduction>
             <mechanicalElasticity>1.0</mechanicalElasticity>
-            <!-- hardwareInterface>PositionJointInterface</hardwareInterface -->
-            <hardwareInterface>EffortJointInterface</hardwareInterface>
+            <!--hardwareInterface>hardware_interface/PositionJointInterface</hardwareInterface-->
+            <hardwareInterface>${Interface10}</hardwareInterface>
           </joint>
           <joint name="${name}_ring_outer_joint">
@@ -263,6 +279,6 @@
             <mechanicalReduction>1.0</mechanicalReduction>
             <mechanicalElasticity>1.0</mechanicalElasticity>
-            <!-- hardwareInterface>PositionJointInterface</hardwareInterface -->
-            <hardwareInterface>EffortJointInterface</hardwareInterface>
+            <!--hardwareInterface>hardware_interface/PositionJointInterface</hardwareInterface-->
+            <hardwareInterface>${Interface10}</hardwareInterface>
           </joint>
           <joint name="${name}_little_abd_joint">
@@ -271,6 +287,6 @@
             <mechanicalReduction>0.4</mechanicalReduction>
             <mechanicalElasticity>1.0</mechanicalElasticity>
-            <!-- hardwareInterface>PositionJointInterface</hardwareInterface -->
-            <hardwareInterface>EffortJointInterface</hardwareInterface>
+            <!--hardwareInterface>hardware_interface/PositionJointInterface</hardwareInterface-->
+            <hardwareInterface>${Interface10}</hardwareInterface>
           </joint>
           <joint name="${name}_little_inner_joint">
@@ -279,6 +295,6 @@
             <mechanicalReduction>1.0</mechanicalReduction>
             <mechanicalElasticity>1.0</mechanicalElasticity>
-            <!-- hardwareInterface>PositionJointInterface</hardwareInterface -->
-            <hardwareInterface>EffortJointInterface</hardwareInterface>
+            <!--hardwareInterface>hardware_interface/PositionJointInterface</hardwareInterface-->
+            <hardwareInterface>${Interface10}</hardwareInterface>
           </joint>
           <joint name="${name}_little_middle_joint">
@@ -287,6 +303,6 @@
             <mechanicalReduction>1.0</mechanicalReduction>
             <mechanicalElasticity>1.0</mechanicalElasticity>
-            <!-- hardwareInterface>PositionJointInterface</hardwareInterface -->
-            <hardwareInterface>EffortJointInterface</hardwareInterface>
+            <!--hardwareInterface>hardware_interface/PositionJointInterface</hardwareInterface-->
+            <hardwareInterface>${Interface10}</hardwareInterface>
           </joint>
           <joint name="${name}_little_outer_joint">
@@ -295,6 +311,6 @@
             <mechanicalReduction>1.0</mechanicalReduction>
             <mechanicalElasticity>1.0</mechanicalElasticity>
-            <!-- hardwareInterface>PositionJointInterface</hardwareInterface -->
-            <hardwareInterface>EffortJointInterface</hardwareInterface>
+            <!--hardwareInterface>hardware_interface/PositionJointInterface</hardwareInterface-->
+            <hardwareInterface>${Interface10}</hardwareInterface>
           </joint>
           <!-- IMPORTANT: if you change the elasticity or reduction at the joints, this value must be calibrated again to
