Commit message: sensorised pisa hand

File: soft_hand_description/model/soft_hand.transmission.xacro (robot description, xacro)
@@ -2,6 +2,6 @@
 <robot name="robot" xmlns:xacro="http://www.ros.org/wiki/xacro">
     <xacro:property name="Interface30" value="hardware_interface/PositionJointInterface"/>
-		<xacro:property name="Interface10" value="hardware_interface/PositionJointInterface"/>
-    <xacro:property name="Interface40" value="hardware_interface/EffortJointInterface"/>
+		<xacro:property name="Interface40" value="hardware_interface/PositionJointInterface"/>
+    <xacro:property name="Interface10" value="hardware_interface/EffortJointInterface"/>
     <xacro:macro name="finger_transmission" params="name finger">
         <transmission name="${name}_${finger}_abd_trans">
